File: DE0NanoShield/KiCad Workspace/DE0NanoShield.kicad_sch (KiCad schematic)
At the start: 0 parts

Commit message: test2
Parts:
- added SW?: SW_Push, symbol Switch:SW_Push
Changed lines of the file:
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@@
 (kicad_sch (version 20211123) (generator eeschema)
   (paper "A4")
-  (symbol (lib_id "power:+1V1") (at 138.43 90.17 0) (unit 1)
+  (symbol (lib_id "Switch:SW_Push") (at 38.1 24.13 0) (unit 1)
     (in_bom yes) (on_board yes) (fields_autoplaced)
-    (property "Reference" "#PWR?" (id 0) (at 138.43 93.98 0)
+    (property "Reference" "SW?" (id 0) (at 38.1 16.51 0))
+    (property "Value" "SW_Push" (id 1) (at 38.1 19.05 0))
+    (property "Footprint" "" (id 2) (at 38.1 19.05 0)
       (effects (font (size 1.27 1.27)) hide)
     )
-    (property "Value" "+1V1" (id 1) (at 138.43 85.09 0))
-    (property "Footprint" "" (id 2) (at 138.43 90.17 0)
-      (effects (font (size 1.27 1.27)) hide)
-    )
-    (property "Datasheet" "" (id 3) (at 138.43 90.17 0)
+    (property "Datasheet" "~" (id 3) (at 38.1 19.05 0)
       (effects (font (size 1.27 1.27)) hide)
     )
     (pin "1")
+    (pin "2")
   )
   (sheet_instances
@@
   )
   (symbol_instances
-    (path "/8de2d84c-ff45-4d4f-bc49-c166f6ae6b91"
-      (reference "#PWR?") (unit 1) (value "+1V1") (footprint "")
+    (path "/0839ce8d-bc94-4a18-9387-0ce4b277e1aa"
+      (reference "SW?") (unit 1) (value "SW_Push") (footprint "")
     )
   )

Commit message: ,
Parts:
- added SW? (x6): SW_SPDT, symbol Switch:SW_SPDT
- added SW? (x3): SW_Push, symbol Switch:SW_Push
Other:
- moved on the sheet: SW?
Changed lines of the file:
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@@
 (kicad_sch (version 20211123) (generator eeschema)
   (paper "A4")
-  (symbol (lib_id "Switch:SW_Push") (at 38.1 24.13 0) (unit 1)
+  (symbol (lib_id "Switch:SW_Push") (at 33.02 38.1 0) (unit 1)
     (in_bom yes) (on_board yes) (fields_autoplaced)
-    (property "Reference" "SW?" (id 0) (at 38.1 16.51 0))
-    (property "Value" "SW_Push" (id 1) (at 38.1 19.05 0))
-    (property "Footprint" "" (id 2) (at 38.1 19.05 0)
+    (property "Reference" "SW?" (id 0) (at 33.02 30.48 0))
+    (property "Value" "SW_Push" (id 1) (at 33.02 33.02 0))
+    (property "Footprint" "" (id 2) (at 33.02 33.02 0)
       (effects (font (size 1.27 1.27)) hide)
     )
-    (property "Datasheet" "~" (id 3) (at 38.1 19.05 0)
+    (property "Datasheet" "~" (id 3) (at 33.02 33.02 0)
       (effects (font (size 1.27 1.27)) hide)
     )
     (pin "1")
     (pin "2")
+  )
+  (symbol (lib_id "Switch:SW_SPDT") (at 71.12 58.42 0) (unit 1)
+    (in_bom yes) (on_board yes) (fields_autoplaced)
+    (property "Reference" "SW?" (id 0) (at 71.12 50.8 0))
+    (property "Value" "SW_SPDT" (id 1) (at 71.12 53.34 0))
+    (property "Footprint" "" (id 2) (at 71.12 58.42 0)
+      (effects (font (size 1.27 1.27)) hide)
+    )
+    (property "Datasheet" "~" (id 3) (at 71.12 58.42 0)
+      (effects (font (size 1.27 1.27)) hide)
+    )
+    (pin "1")
+    (pin "2")
+    (pin "3")
+  )
+  (symbol (lib_id "Switch:SW_SPDT") (at 87.63 58.42 0) (unit 1)
+    (in_bom yes) (on_board yes) (fields_autoplaced)
+    (property "Reference" "SW?" (id 0) (at 87.63 50.8 0))
+    (property "Value" "SW_SPDT" (id 1) (at 87.63 53.34 0))
+    (property "Footprint" "" (id 2) (at 87.63 58.42 0)
+      (effects (font (size 1.27 1.27)) hide)
+    )
+    (property "Datasheet" "~" (id 3) (at 87.63 58.42 0)
+      (effects (font (size 1.27 1.27)) hide)
+    )
+    (pin "1")
+    (pin "2")
+    (pin "3")
+  )
+  (symbol (lib_id "Switch:SW_SPDT") (at 124.46 58.42 0) (unit 1)
+    (in_bom yes) (on_board yes) (fields_autoplaced)
+    (property "Reference" "SW?" (id 0) (at 124.46 50.8 0))
+    (property "Value" "SW_SPDT" (id 1) (at 124.46 53.34 0))
+    (property "Footprint" "" (id 2) (at 124.46 58.42 0)
+      (effects (font (size 1.27 1.27)) hide)
+    )
+    (property "Datasheet" "~" (id 3) (at 124.46 58.42 0)
+      (effects (font (size 1.27 1.27)) hide)
+    )
+    (pin "1")
+    (pin "2")
+    (pin "3")
+  )
+  (symbol (lib_id "Switch:SW_SPDT") (at 33.02 58.42 0) (unit 1)
+    (in_bom yes) (on_board yes) (fields_autoplaced)
+    (property "Reference" "SW?" (id 0) (at 33.02 50.8 0))
+    (property "Value" "SW_SPDT" (id 1) (at 33.02 53.34 0))
+    (property "Footprint" "" (id 2) (at 33.02 58.42 0)
+      (effects (font (size 1.27 1.27)) hide)
+    )
+    (property "Datasheet" "~" (id 3) (at 33.02 58.42 0)
+      (effects (font (size 1.27 1.27)) hide)
+    )
+    (pin "1")
+    (pin "2")
+    (pin "3")
+  )
+  (symbol (lib_id "Switch:SW_Push") (at 92.71 38.1 0) (unit 1)
+    (in_bom yes) (on_board yes) (fields_autoplaced)
+    (property "Reference" "SW?" (id 0) (at 92.71 30.48 0))
+    (property "Value" "SW_Push" (id 1) (at 92.71 33.02 0))
+    (property "Footprint" "" (id 2) (at 92.71 33.02 0)
+      (effects (font (size 1.27 1.27)) hide)
+    )
+    (property "Datasheet" "~" (id 3) (at 92.71 33.02 0)
+      (effects (font (size 1.27 1.27)) hide)
+    )
+    (pin "1")
+    (pin "2")
+  )
+  (symbol (lib_id "Switch:SW_SPDT") (at 106.68 58.42 0) (unit 1)
+    (in_bom yes) (on_board yes) (fields_autoplaced)
+    (property "Reference" "SW?" (id 0) (at 106.68 50.8 0))
+    (property "Value" "SW_SPDT" (id 1) (at 106.68 53.34 0))
+    (property "Footprint" "" (id 2) (at 106.68 58.42 0)
+      (effects (font (size 1.27 1.27)) hide)
+    )
+    (property "Datasheet" "~" (id 3) (at 106.68 58.42 0)
+      (effects (font (size 1.27 1.27)) hide)
+    )
+    (pin "1")
+    (pin "2")
+    (pin "3")
+  )
+  (symbol (lib_id "Switch:SW_Push") (at 73.66 38.1 0) (unit 1)
+    (in_bom yes) (on_board yes) (fields_autoplaced)
+    (property "Reference" "SW?" (id 0) (at 73.66 30.48 0))
+    (property "Value" "SW_Push" (id 1) (at 73.66 33.02 0))
+    (property "Footprint" "" (id 2) (at 73.66 33.02 0)
+      (effects (font (size 1.27 1.27)) hide)
+    )
+    (property "Datasheet" "~" (id 3) (at 73.66 33.02 0)
+      (effects (font (size 1.27 1.27)) hide)
+    )
+    (pin "1")
+    (pin "2")
+  )
+  (symbol (lib_id "Switch:SW_Push") (at 54.61 38.1 0) (unit 1)
+    (in_bom yes) (on_board yes) (fields_autoplaced)
+    (property "Reference" "SW?" (id 0) (at 54.61 30.48 0))
+    (property "Value" "SW_Push" (id 1) (at 54.61 33.02 0))
+    (property "Footprint" "" (id 2) (at 54.61 33.02 0)
+      (effects (font (size 1.27 1.27)) hide)
+    )
+    (property "Datasheet" "~" (id 3) (at 54.61 33.02 0)
+      (effects (font (size 1.27 1.27)) hide)
+    )
+    (pin "1")
+    (pin "2")
+  )
+  (symbol (lib_id "Switch:SW_SPDT") (at 53.34 58.42 0) (unit 1)
+    (in_bom yes) (on_board yes) (fields_autoplaced)
+    (property "Reference" "SW?" (id 0) (at 53.34 50.8 0))
+    (property "Value" "SW_SPDT" (id 1) (at 53.34 53.34 0))
+    (property "Footprint" "" (id 2) (at 53.34 58.42 0)
+      (effects (font (size 1.27 1.27)) hide)
+    )
+    (property "Datasheet" "~" (id 3) (at 53.34 58.42 0)
+      (effects (font (size 1.27 1.27)) hide)
+    )
+    (pin "1")
+    (pin "2")
+    (pin "3")
   )
   (sheet_instances
@@
       (reference "SW?") (unit 1) (value "SW_Push") (footprint "")
     )
+    (path "/2ad47cb7-2e83-46dc-8238-c822230299ef"
+      (reference "SW?") (unit 1) (value "SW_SPDT") (footprint "")
+    )
+    (path "/3d1134d0-6c97-4810-8ed8-3e980e55edea"
+      (reference "SW?") (unit 1) (value "SW_SPDT") (footprint "")
+    )
+    (path "/55cc41bb-59f6-4bfb-9f86-63b8f1c7cd87"
+      (reference "SW?") (unit 1) (value "SW_SPDT") (footprint "")
+    )
+    (path "/5cece746-e816-46a9-947d-0c591d8774f9"
+      (reference "SW?") (unit 1) (value "SW_SPDT") (footprint "")
+    )
+    (path "/7e5cbe65-fc5e-45b5-85c1-bde34d1f9056"
+      (reference "SW?") (unit 1) (value "SW_Push") (footprint "")
+    )
+    (path "/8429cba8-519f-40a9-8cd5-cac7da4ba07e"
+      (reference "SW?") (unit 1) (value "SW_SPDT") (footprint "")
+    )
+    (path "/a0ed2662-e29b-4edc-8d41-dd4e00e3476a"
+      (reference "SW?") (unit 1) (value "SW_Push") (footprint "")
+    )
+    (path "/a756a3d8-e7f6-433b-b40a-4f16e0acf771"
+      (reference "SW?") (unit 1) (value "SW_Push") (footprint "")
+    )
+    (path "/aff7510b-1d93-4425-867a-b9b2e0c29065"
+      (reference "SW?") (unit 1) (value "SW_SPDT") (footprint "")
+    )
   )

Commit message: summary
Parts:
- added J?: Conn_01x16_Male, symbol Connector:Conn_01x16_Male
- added U?: LTC-4627JD, Display_7Segment:LTC-4627Jx, symbol Display_Character:LTC-4627JD
Changed lines of the file:
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@@
     (pin "3")
+  )
+  (symbol (lib_id "Display_Character:LTC-4627JD") (at 262.89 31.75 0) (unit 1)
+    (in_bom yes) (on_board yes) (fields_autoplaced)
+    (property "Reference" "U?" (id 0) (at 262.89 15.24 0))
+    (property "Value" "LTC-4627JD" (id 1) (at 262.89 17.78 0))
+    (property "Footprint" "Display_7Segment:LTC-4627Jx" (id 2) (at 262.89 44.45 0)
+      (effects (font (size 1.27 1.27)) hide)
+    )
+    (property "Datasheet" "http://optoelectronics.liteon.com/upload/download/DS30-2001-093/LTC-4627JD.pdf" (id 3) (at 252.73 31.75 0)
+      (effects (font (size 1.27 1.27)) hide)
+    )
+    (pin "1")
+    (pin "11")
+    (pin "13")
+    (pin "14")
+    (pin "15")
+    (pin "16")
+    (pin "2")
+    (pin "3")
+    (pin "4")
+    (pin "5")
+    (pin "6")
+    (pin "7")
+    (pin "8")
+    (pin "9")
   )
   (symbol (lib_id "Switch:SW_Push") (at 73.66 38.1 0) (unit 1)
@@
     (pin "3")
   )
+  (symbol (lib_id "Connector:Conn_01x16_Male") (at 265.43 72.39 0) (unit 1)
+    (in_bom yes) (on_board yes) (fields_autoplaced)
+    (property "Reference" "J?" (id 0) (at 266.065 49.53 0))
+    (property "Value" "Conn_01x16_Male" (id 1) (at 266.065 52.07 0))
+    (property "Footprint" "" (id 2) (at 265.43 72.39 0)
+      (effects (font (size 1.27 1.27)) hide)
+    )
+    (property "Datasheet" "~" (id 3) (at 265.43 72.39 0)
+      (effects (font (size 1.27 1.27)) hide)
+    )
+    (pin "1")
+    (pin "10")
+    (pin "11")
+    (pin "12")
+    (pin "13")
+    (pin "14")
+    (pin "15")
+    (pin "16")
+    (pin "2")
+    (pin "3")
+    (pin "4")
+    (pin "5")
+    (pin "6")
+    (pin "7")
+    (pin "8")
+    (pin "9")
+  )
   (sheet_instances
     (path "/" (page "1"))
   )
   (symbol_instances
+    (path "/f701839a-88fc-4935-befa-f16fe6ff7b7e"
+      (reference "J?") (unit 1) (value "Conn_01x16_Male") (footprint "")
+    )
     (path "/0839ce8d-bc94-4a18-9387-0ce4b277e1aa"
       (reference "SW?") (unit 1) (value "SW_Push") (footprint "")
@@
       (reference "SW?") (unit 1) (value "SW_SPDT") (footprint "")
     )
+    (path "/856f7da1-1617-4555-b513-8ce6a5afc8b3"
+      (reference "U?") (unit 1) (value "LTC-4627JD") (footprint "Display_7Segment:LTC-4627Jx")
+    )
   )

Commit message: added more symbols
Parts:
- added D? (x6): LED, symbol Device:LED
- added J? (x2): Conn_01x40_MountingPin, symbol Connector_Generic_MountingPin:Conn_01x40_MountingPin
- added J?: RJ45_Bel_SI-60062-F, Connector_RJ:RJ45_Bel_SI-60062-F, symbol Connector:RJ45_Bel_SI-60062-F
- added J?: SD_Card, symbol Connector:SD_Card
- added J?: Conn_01x08, symbol Connector_Generic:Conn_01x08
- added J?: USB_B_Micro, symbol Connector:USB_B_Micro
- added J?: Conn_01x06, symbol Connector_Generic:Conn_01x06
Other:
- moved on the sheet: J?, SW?, U?
