File: DE0NanoShield/KiCad Workspace/DE0NanoShield.kicad_sch (KiCad schematic)
At the start: 76 parts, among them J1 Conn_01x40_MountingPin, J2 Conn_01x40_MountingPin, J3 Conn_01x16_Male, J4 Conn_01x06_MountingPin, J5 Conn_01x06_MountingPin, J6 Conn_01x06_MountingPin, J7 Conn_01x12_MountingPin, J8 Conn_01x08_Female, SW1 SW_SPDT, SW10 SW_SPDT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

Commit message: Added missing footprints
Parts:
- FL1: footprint BEADC1005X55N -> Additional Footprints and Symbols:BEADC1005X55N
- U2: footprint SOP50P490X110-10N -> Additional Footprints and Symbols:SOP50P490X110-10N
Changed lines of the file:
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@@
     (property "Reference" "U2" (id 0) (at 289.052 260.604 0))
     (property "Value" "CS4344-CZZ" (id 1) (at 289.052 263.144 0))
-    (property "Footprint" "SOP50P490X110-10N" (id 2) (at 289.052 278.384 0)
+    (property "Footprint" "Additional Footprints and Symbols:SOP50P490X110-10N" (id 2) (at 289.052 278.384 0)
       (effects (font (size 1.27 1.27)) (justify left bottom) hide)
     )
@@
     (property "Reference" "FL1" (id 0) (at 236.22 275.844 0))
     (property "Value" "600" (id 1) (at 236.22 278.384 0))
-    (property "Footprint" "BEADC1005X55N" (id 2) (at 237.49 283.464 0)
+    (property "Footprint" "Additional Footprints and Symbols:BEADC1005X55N" (id 2) (at 237.49 283.464 0)
       (effects (font (size 1.27 1.27)) (justify left bottom) hide)
     )
@@
     )
     (path "/b198605c-23ab-4542-bcca-1318b54a0a97"
-      (reference "FL1") (unit 1) (value "600") (footprint "BEADC1005X55N")
+      (reference "FL1") (unit 1) (value "600") (footprint "Additional Footprints and Symbols:BEADC1005X55N")
     )
     (path "/3737b56d-25ae-4564-bb74-94ce2d17ace8"
@@
     )
     (path "/14c5a91a-78b9-4906-ad0e-76dc562e24aa"
-      (reference "U2") (unit 1) (value "CS4344-CZZ") (footprint "SOP50P490X110-10N")
-    )
-  )
+      (reference "U2") (unit 1) (value "CS4344-CZZ") (footprint "Additional Footprints and Symbols:SOP50P490X110-10N")
+    )
+  )

Commit message: finished schematic completely all footprints assigned
Parts:
- SW11: footprint (none) -> Rotary_Encoder:RotaryEncoder_Alps_EC11E-Switch_Vertical_H20mm
Changed lines of the file:
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@@
     (property "Reference" "SW11" (id 0) (at 129.794 275.59 0))
     (property "Value" "RotaryEncoder_Switch" (id 1) (at 129.794 278.13 0))
-    (property "Footprint" "" (id 2) (at 125.984 281.432 0)
+    (property "Footprint" "Rotary_Encoder:RotaryEncoder_Alps_EC11E-Switch_Vertical_H20mm" (id 2) (at 125.984 281.432 0)
       (effects (font (size 1.27 1.27)) hide)
     )
@@
     )
     (path "/9464acfd-8c29-443e-81cb-e5498b72dd14"
-      (reference "SW11") (unit 1) (value "RotaryEncoder_Switch") (footprint "")
+      (reference "SW11") (unit 1) (value "RotaryEncoder_Switch") (footprint "Rotary_Encoder:RotaryEncoder_Alps_EC11E-Switch_Vertical_H20mm")
     )
     (path "/e2228ec7-985b-43b9-8d7e-0bef3e2c842e"
